Commit message: docs: Add README and demo image, fix Husky URDF base_footprint joint, and update launch configurations.

File: urdf/husky.urdf.xacro (robot description, xacro)
@@ -72,7 +72,7 @@
   <link name="base_footprint"/>
   <joint name="base_footprint_joint" type="fixed">
-    <origin xyz="0 0 ${wheel_vertical_offset - wheel_radius}" rpy="0 0 0" />
-    <parent link="base_link" />
-    <child link="base_footprint" />
+    <parent link="base_footprint"/>
+    <child link="base_link"/>
+    <origin xyz="0 0 ${-wheel_vertical_offset + wheel_radius}" rpy="0 0 0"/>
   </joint>
   <!-- Inertial link stores the robot's inertial information -->
